File: OmegaKit_Junior/OmegaKit_Junior.kicad_pcb (KiCad board)
At the start: 2 copper layers, 83.5 x 37 mm, 19 parts, among them SW1 SW_CK_OS102011MS2Q, U1 TSOP1838

Commit message: Novo .step placa juniores
Parts:
- added ?: , , F.Cu at (109.5, 57.0)
- added ?: , , F.Cu at (109.5, 90.0)
- added ?: , , F.Cu at (189.0, 57.0)
- turned RET to 180 degrees

Commit message: ✨ feat: atualização de todos os arquivps faltantes
Parts:
- renumbered TB6612FNG1 to TB6612FNG
Other:
- board text added: "10/08/2025"
Changed lines of the file:
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@@
 		(descr "Through hole straight socket strip, 1x08, 2.54mm pitch, single row (from Kicad 4.0.7), script generated")
 		(tags "Through hole socket strip THT 1x08 2.54mm single row")
-		(property "Reference" "TB6612FNG1"
+		(property "Reference" "TB6612FNG"
 			(at 7.5 9.2 90)
 			(layer "F.SilkS")
@@
 			(unlocked yes)
 			(layer "F.SilkS")
+			(hide yes)
 			(effects
 				(font
@@
 		)
 	)
+	(gr_text "10/08/2025"
+		(at 139.5 73.5 90)
+		(layer "F.SilkS")
+		(effects
+			(font
+				(size 1 1)
+				(thickness 0.1)
+			)
+			(justify left bottom)
+		)
+	)
