File: OmegaKit_ESP_Embarcado_Simplificado/OmegaKit_ESP_Embarcado_Simplificado.kicad_pcb (KiCad board)
At the start: 2 copper layers, 76.5 x 36.5 mm, 49 parts, among them J13 Conn_01x02_Socket, J2 MOTOR_B, J5 MOTOR_A, Q25 QTR_1, Q26 QTR_2, SW1 TS-1088-AR02016, SW2 TS-1088-AR02016, SW3 SS-12D10G5, U1 AMS1117-5.0, U2 TB6612FNG, U3 ESP32-WROOM-32, U5 AMS1117-3.3

Commit message: ✨ feat: atualização de todos os arquivps faltantes
Parts:
- removed R2: 100Ohm, Resistor_SMD:R_0805_2012Metric_Pad1.20x1.40mm_HandSolder
- added C6: 100 nF, Capacitor_SMD:C_0201_0603Metric_Pad0.64x0.40mm_HandSolder, F.Cu at (102.1, 59.0)
- renumbered Q25 to Q34, Q26 to Q35, S27 to S25, S32 to S26, S33 to S27, S34 to S32, S35 to S33
Connections:
- SW2 pad 1: Net-(R2-Pad2) -> BOOT
- U3 pad 10: QTR1 -> SENSOR1
- U3 pad 11: QTR2 -> SENSOR2
- U3 pad 12: SENSOR1 -> SENSOR3
- U3 pad 6: SENSOR4 -> QTR1
- U3 pad 7: SENSOR5 -> QTR2
- U3 pad 8: SENSOR2 -> SENSOR4
- U3 pad 9: SENSOR3 -> SENSOR5
Routing:
- net SENSOR3: track 53.1 -> 48.3 mm
- net QTR2: track 6.73 -> 11.5 mm
- net QTR1: track 10.9 -> 6.18 mm
- net SENSOR2: track 46.6 -> 42.7 mm
- net Net-(R2-Pad2): track 3.71 -> 0.00 mm
- net SENSOR5: track 36.7 -> 33.8 mm
- net SENSOR4: track 28.5 -> 25.6 mm
- net SENSOR1: track 57.1 -> 58.6 mm
- net BIN1: track 57.2 -> 56.2 mm
Other:
- board text added: "18/02/2026"
- board text added: "優勝まで"
