File: OmegaKit_ESP_Embarcado_Simplificado/OmegaKit_ESP_Embarcado_Simplificado.kicad_sch (KiCad schematic)
At the start: 45 parts, among them J13 Conn_01x02_Socket, J2 MOTOR_B, J5 MOTOR_A, Q25 QTR_1, Q26 QTR_2, SW1 TS-1088-AR02016, SW2 TS-1088-AR02016, SW3 SS-12D10G5, U1 AMS1117-5.0, U2 TB6612FNG, U3 ESP32-WROOM-32, U5 AMS1117-3.3

Commit message: ✨ feat: atualização de todos os arquivps faltantes
Parts:
- removed R2: 100Ohm, Resistor_SMD:R_0805_2012Metric_Pad1.20x1.40mm_HandSolder, symbol Device:R
- added C6: 100 nF, Capacitor_SMD:C_0201_0603Metric_Pad0.64x0.40mm_HandSolder, symbol Device:C_US
- renumbered Q25 to Q34, Q26 to Q35, S27 to S25, S32 to S26, S33 to S27, S34 to S32, S35 to S33
Connections:
- net BOOT: now also SW2.1, C6.1
- net GND: now also C6.2
- net QTR1: now also U3.6 (IO34); no longer U3.10 (IO25)
- net QTR2: now also U3.7 (IO35); no longer U3.11 (IO26)
- net SENSOR1: now also U3.10 (IO25); no longer U3.12 (IO27)
- net SENSOR2: now also U3.11 (IO26); no longer U3.8 (IO32)
- net SENSOR3: now also U3.12 (IO27); no longer U3.9 (IO33)
- net SENSOR4: now also U3.8 (IO32); no longer U3.6 (IO34)
- net SENSOR5: now also U3.9 (IO33); no longer U3.7 (IO35)
