File: OmegaKit_RZ60/OmegaKit_RZ60.kicad_sch (KiCad schematic)
At the start: 19 parts, among them SW1 SW_CK_OS102011MS2Q, U1 AMS1117-5.0

Commit message: ✨ feat: atualização de todos os arquivps faltantes
Connections:
- net VCC: no longer IR17.3 (VCC), TB6612FNG1.2 (VCC)
- net V_REG: now also IR17.3 (VCC), TB6612FNG1.2 (VCC)
Changed lines of the file:
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@@
 	(wire
 		(pts
-			(xy 241.3 86.36) (xy 245.11 86.36)
+			(xy 241.3 86.36) (xy 248.92 86.36)
 		)
 		(stroke
@@
 		)
 	)
-	(label "VCC"
+	(label "V_REG"
 		(at 127 116.84 0)
 		(effects
@@
 		)
 	)
-	(label "VCC"
-		(at 245.11 86.36 180)
-		(effects
-			(font
+	(label "V_REG"
+		(at 248.92 86.36 180)
+		(effects
+			(font
